File: src/robot-power-pcb.kicad_pcb (KiCad board)
At the start: 2 copper layers, 93 x 84.5 mm, 6 parts, among them J1 PWR Supply Port, J2 Arduino Terminal, J3 Motor 2 Terminal, J4 Motor 1 Terminal, U1 L2596S, U2 Mini PWM Controller

Commit message: Update of project
Routing:
- net GND: track 0.41 -> 172.5 mm
Changed lines of the file:
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@@
+	)
+	(segment
+		(start 128.2 67.7)
+		(end 133.9 62)
+		(width 0.2)
+		(layer "F.Cu")
+		(net 1)
+	)
+	(segment
+		(start 145.35 86.862)
+		(end 145.35 85.9)
+		(width 0.2)
+		(layer "F.Cu")
+		(net 1)
+	)
+	(segment
+		(start 131.5 78.2)
+		(end 128.2 74.9)
+		(width 0.2)
+		(layer "F.Cu")
+		(net 1)
+	)
+	(segment
+		(start 195.549335 89)
+		(end 147.488 89)
+		(width 0.2)
+		(layer "F.Cu")
+		(net 1)
+	)
+	(segment
+		(start 208.5 73.665)
+		(end 208.5 76.049335)
+		(width 0.2)
+		(layer "F.Cu")
+		(net 1)
+	)
+	(segment
+		(start 196.835 62)
+		(end 208.5 73.665)
+		(width 0.2)
+		(layer "F.Cu")
+		(net 1)
+	)
+	(segment
+		(start 133.9 62)
+		(end 196.835 62)
+		(width 0.2)
+		(layer "F.Cu")
+		(net 1)
+	)
+	(segment
+		(start 208.5 76.049335)
+		(end 195.549335 89)
+		(width 0.2)
+		(layer "F.Cu")
+		(net 1)
 	)
 	(segment
@@
 		(width 0.2)
 		(layer "F.Cu")
+		(net 1)
+	)
+	(segment
+		(start 128.2 74.9)
+		(end 128.2 67.7)
+		(width 0.2)
+		(layer "F.Cu")
+		(net 1)
+	)
+	(segment
+		(start 147.488 89)
+		(end 145.35 86.862)
+		(width 0.2)
+		(layer "F.Cu")
